File: epaper.kicad_sch (KiCad schematic)
At the start: 19 parts, among them J10 E-Paper, Q3 AP2302B

Commit message: Fill out BOM, add labels to PCB
Parts:
- C13, C14, C16, C17, C18, C19, C20, C21: LCSC (none) -> C5199872
- C15: LCSC (none) -> C69335
- C22: LCSC (none) -> C1623
- R34: LCSC (none) -> C25101
- R35: LCSC (none) -> C25741
Changed lines of the file:
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@@
 			)
 		)
-		(property "Datasheet" "https://datasheet.lcsc.com/lcsc/2304140030_CCTC-TCC0805X7R105M500FT_C376929.pdf"
+		(property "Datasheet" "https://datasheet.lcsc.com/lcsc/2304140030_Samsung-Electro-Mechanics-CL05A105KQ5NNNC_C107372.pdf"
 			(at 114.3 128.27 0)
 			(effects
@@
 			)
 		)
-		(property "LCSC" ""
+		(property "LCSC" "C5199872"
 			(at 114.3 128.27 0)
 			(effects
@@
 			)
 		)
-		(property "Datasheet" "https://datasheet.lcsc.com/lcsc/2304140030_CCTC-TCC0805X7R105M500FT_C376929.pdf"
+		(property "Datasheet" "https://datasheet.lcsc.com/lcsc/2304140030_Samsung-Electro-Mechanics-CL05A105KQ5NNNC_C107372.pdf"
 			(at 158.75 128.27 0)
 			(effects
@@
 			)
 		)
-		(property "LCSC" ""
+		(property "LCSC" "C5199872"
 			(at 158.75 128.27 0)
 			(effects
@@
 			)
 		)
-		(property "Datasheet" "https://datasheet.lcsc.com/lcsc/2308241947_FOJAN-FRC0805J104-TS_C2907293.pdf"
+		(property "Datasheet" "https://www.lcsc.com/product-detail/Chip-Resistor-Surface-Mount_UNI-ROYAL-Uniroyal-Elec-0402WGF1003TCE_C25741.html"
 			(at 114.3 72.39 0)
 			(effects
@@
 			)
 		)
-		(property "LCSC" ""
+		(property "LCSC" "C25741"
 			(at 114.3 72.39 0)
 			(effects
@@
 			)
 		)
-		(property "Datasheet" "https://datasheet.lcsc.com/lcsc/2304140030_CCTC-TCC0805X7R105M500FT_C376929.pdf"
+		(property "Datasheet" "https://datasheet.lcsc.com/lcsc/2304140030_Samsung-Electro-Mechanics-CL05A105KQ5NNNC_C107372.pdf"
 			(at 132.08 128.27 0)
 			(effects
@@
 			)
 		)
-		(property "LCSC" ""
+		(property "LCSC" "C5199872"
 			(at 132.08 128.27 0)
 			(effects
@@
 			)
 		)
-		(property "Datasheet" "https://datasheet.lcsc.com/lcsc/2304140030_CCTC-TCC0805X7R105M500FT_C376929.pdf"
+		(property "Datasheet" "https://datasheet.lcsc.com/lcsc/2304140030_Samsung-Electro-Mechanics-CL05A105KQ5NNNC_C107372.pdf"
 			(at 91.44 130.81 0)
 			(effects
@@
 			)
 		)
-		(property "LCSC" ""
+		(property "LCSC" "C5199872"
 			(at 91.44 130.81 0)
 			(effects
@@
 			)
 		)
-		(property "Datasheet" "https://datasheet.lcsc.com/lcsc/2304140030_CCTC-TCC0805X7R105M500FT_C376929.pdf"
+		(property "Datasheet" "https://datasheet.lcsc.com/lcsc/2304140030_Samsung-Electro-Mechanics-CL05A105KQ5NNNC_C107372.pdf"
 			(at 149.86 128.27 0)
 			(effects
@@
 			)
 		)
-		(property "LCSC" ""
+		(property "LCSC" "C5199872"
 			(at 149.86 128.27 0)
 			(effects
@@
 			)
 		)
-		(property "Datasheet" "https://datasheet.lcsc.com/lcsc/2304140030_CCTC-TCC0805X7R105M500FT_C376929.pdf"
+		(property "Datasheet" "https://datasheet.lcsc.com/lcsc/2304140030_Samsung-Electro-Mechanics-CL05A105KQ5NNNC_C107372.pdf"
 			(at 91.44 115.57 0)
 			(effects
@@
 			)
 		)
-		(property "LCSC" ""
+		(property "LCSC" "C5199872"
 			(at 91.44 115.57 0)
 			(effects
@@
 			)
 		)
-		(property "Datasheet" "https://datasheet.lcsc.com/lcsc/2111172030_Samwha-Capacitor-CS2012X5R475K250NRE_C2918489.pdf"
+		(property "Datasheet" "https://datasheet.lcsc.com/lcsc/1810261513_Samsung-Electro-Mechanics-CL10A475KA8NQNC_C69335.pdf"
 			(at 77.47 72.39 0)
 			(effects
@@
 			)
 		)
-		(property "LCSC" ""
+		(property "LCSC" "C69335"
 			(at 77.47 72.39 0)
 			(effects
@@
 			)
 		)
-		(property "Datasheet" "https://datasheet.lcsc.com/lcsc/2308241947_FOJAN-FRC0805J270-TS_C2907314.pdf"
+		(property "Datasheet" "https://www.lcsc.com/product-detail/Chip-Resistor-Surface-Mount_UNI-ROYAL-Uniroyal-Elec-0402WGF220KTCE_C25101.html"
 			(at 106.68 72.39 0)
 			(effects
@@
 			)
 		)
-		(property "LCSC" ""
+		(property "LCSC" "C25101"
 			(at 106.68 72.39 0)
 			(effects
@@
 			)
 		)
-		(property "Datasheet" "https://datasheet.lcsc.com/lcsc/2304140030_CCTC-TCC0805X7R105M500FT_C376929.pdf"
+		(property "Datasheet" "https://datasheet.lcsc.com/lcsc/2304140030_Samsung-Electro-Mechanics-CL05A105KQ5NNNC_C107372.pdf"
 			(at 123.19 128.27 0)
 			(effects
@@
 			)
 		)
-		(property "LCSC" ""
+		(property "LCSC" "C5199872"
 			(at 123.19 128.27 0)
 			(effects
@@
 			)
 		)
-		(property "Datasheet" "https://datasheet.lcsc.com/lcsc/2108150230_FH--Guangdong-Fenghua-Advanced-Tech-0805B474K250NT_C2859120.pdf"
+		(property "Datasheet" "https://www.lcsc.com/product-detail/Multilayer-Ceramic-Capacitors-MLCC-SMD-SMT_Samsung-Electro-Mechanics-CL10B474KA8NNNC_C1623.html"
 			(at 167.64 128.27 0)
 			(effects
@@
 			)
 		)
-		(property "LCSC" ""
+		(property "LCSC" "C1623"
 			(at 167.64 128.27 0)
 			(effects
@@
 			)
 		)
-		(property "Datasheet" "https://datasheet.lcsc.com/lcsc/2304140030_CCTC-TCC0805X7R105M500FT_C376929.pdf"
+		(property "Datasheet" "https://datasheet.lcsc.com/lcsc/2304140030_Samsung-Electro-Mechanics-CL05A105KQ5NNNC_C107372.pdf"
 			(at 140.97 128.27 0)
 			(effects
@@
 			)
 		)
-		(property "LCSC" ""
+		(property "LCSC" "C5199872"
 			(at 140.97 128.27 0)
 			(effects

Commit message: Changes for production version
Parts:
- C13, C14, C15, C16, C17, C18, C19, C20, C21, C22: footprint Capacitor_SMD:C_0402_1005Metric -> Capacitor_SMD:C_0603_1608Metric
- R34: footprint Resistor_SMD:R_0402_1005Metric -> Resistor_SMD:R_0805_2012Metric; LCSC C25101 -> C2907304
Changed lines of the file:
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@@
 (kicad_sch
-	(version 20231120)
+	(version 20250114)
 	(generator "eeschema")
-	(generator_version "8.0")
+	(generator_version "9.0")
 	(paper "A4")
 	(title_block
@@
 		(comment 1 "License: CERN Open Hardware Licence Version 2 - Permissive")
 	)
+	(text "VDD"
+		(exclude_from_sim no)
+		(at 167.64 101.6 0)
+		(effects
+			(font
+				(size 1.27 1.27)
+			)
+			(justify left bottom)
+		)
+	)
+	(text "VSS"
+		(exclude_from_sim no)
+		(at 167.64 99.06 0)
+		(effects
+			(font
+				(size 1.27 1.27)
+			)
+			(justify left bottom)
+		)
+	)
+	(text "BS1"
+		(exclude_from_sim no)
+		(at 167.64 76.2 0)
+		(effects
+			(font
+				(size 1.27 1.27)
+			)
+			(justify left bottom)
+		)
+	)
+	(text "VDDIO"
+		(exclude_from_sim no)
+		(at 167.64 93.98 0)
+		(effects
+			(font
+				(size 1.27 1.27)
+			)
+			(justify left bottom)
+		)
+	)
+	(text "VCI"
+		(exclude_from_sim no)
+		(at 167.64 96.52 0)
+		(effects
+			(font
+				(size 1.27 1.27)
+			)
+			(justify left bottom)
+		)
+	)
+	(text "VPP"
+		(exclude_from_sim no)
+		(at 167.64 104.14 0)
+		(effects
+			(font
+				(size 1.27 1.27)
+			)
+			(justify left bottom)
+		)
+	)
 	(junction
 		(at 140.97 96.52)
@@
 		)
 	)
-	(text "VDD"
-		(exclude_from_sim no)
-		(at 167.64 101.6 0)
-		(effects
-			(font
-				(size 1.27 1.27)
-			)
-			(justify left bottom)
-		)
-	)
-	(text "VSS"
-		(exclude_from_sim no)
-		(at 167.64 99.06 0)
-		(effects
-			(font
-				(size 1.27 1.27)
-			)
-			(justify left bottom)
-		)
-	)
-	(text "BS1"
-		(exclude_from_sim no)
-		(at 167.64 76.2 0)
-		(effects
-			(font
-				(size 1.27 1.27)
-			)
-			(justify left bottom)
-		)
-	)
-	(text "VDDIO"
-		(exclude_from_sim no)
-		(at 167.64 93.98 0)
-		(effects
-			(font
-				(size 1.27 1.27)
-			)
-			(justify left bottom)
-		)
-	)
-	(text "VCI"
-		(exclude_from_sim no)
-		(at 167.64 96.52 0)
-		(effects
-			(font
-				(size 1.27 1.27)
-			)
-			(justify left bottom)
-		)
-	)
-	(text "VPP"
-		(exclude_from_sim no)
-		(at 167.64 104.14 0)
-		(effects
-			(font
-				(size 1.27 1.27)
-			)
-			(justify left bottom)
-		)
-	)
 	(label "GDR"
 		(at 167.64 60.96 0)
-		(fields_autoplaced yes)
 		(effects
 			(font
@@
 	(label "PREVGL"
 		(at 167.64 114.3 0)
-		(fields_autoplaced yes)
 		(effects
 			(font
@@
 	(label "VSL"
 		(at 167.64 111.76 0)
-		(fields_autoplaced yes)
 		(effects
 			(font
@@
 	(label "VCOM"
 		(at 167.64 116.84 0)
-		(fields_autoplaced yes)
 		(effects
 			(font
@@
 	(label "VGL"
 		(at 167.64 66.04 0)
-		(fields_autoplaced yes)
 		(effects
 			(font
@@
 	(label "VSH"
 		(at 167.64 106.68 0)
-		(fields_autoplaced yes)
 		(effects
 			(font
@@
 	(label "PREVGH"
 		(at 167.64 109.22 0)
-		(fields_autoplaced yes)
 		(effects
 			(font
@@
 	(label "RESE"
 		(at 167.64 63.5 0)
-		(fields_autoplaced yes)
 		(effects
 			(font
@@
 	(label "VGH"
 		(at 167.64 68.58 0)
-		(fields_autoplaced yes)
 		(effects
 			(font
@@
 		(shape bidirectional)
 		(at 172.72 81.28 180)
-		(fields_autoplaced yes)
 		(effects
 			(font
@@
 		(shape bidirectional)
 		(at 172.72 86.36 180)
-		(fields_autoplaced yes)
 		(effects
 			(font
@@
 		(shape bidirectional)
 		(at 172.72 78.74 180)
-		(fields_autoplaced yes)
 		(effects
 			(font
@@
 		(shape bidirectional)
 		(at 172.72 83.82 180)
-		(fields_autoplaced yes)
 		(effects
 			(font
@@
 		(shape bidirectional)
 		(at 172.72 88.9 180)
-		(fields_autoplaced yes)
 		(effects
 			(font
@@
 		(shape bidirectional)
 		(at 172.72 91.44 180)
-		(fields_autoplaced yes)
 		(effects
 			(font
@@
 			)
 		)
-		(property "Footprint" "Capacitor_SMD:C_0402_1005Metric"
+		(property "Footprint" "Capacitor_SMD:C_0603_1608Metric"
 			(at 113.3348 124.46 0)
 			(effects
@@
 			)
 		)
-		(property "Footprint" "Capacitor_SMD:C_0402_1005Metric"
+		(property "Footprint" "Capacitor_SMD:C_0603_1608Metric"
 			(at 157.7848 124.46 0)
 			(effects
@@
 			)
 		)
-		(property "Footprint" "Capacitor_SMD:C_0402_1005Metric"
+		(property "Footprint" "Capacitor_SMD:C_0603_1608Metric"
 			(at 131.1148 124.46 0)
 			(effects
@@
 			)
 		)
-		(property "Footprint" "Capacitor_SMD:C_0402_1005Metric"
+		(property "Footprint" "Capacitor_SMD:C_0603_1608Metric"
 			(at 87.63 129.8448 0)
 			(effects
@@
 			)
 		)
-		(property "Footprint" "Capacitor_SMD:C_0402_1005Metric"
+		(property "Footprint" "Capacitor_SMD:C_0603_1608Metric"
 			(at 148.8948 124.46 0)
 			(effects
@@
 			)
 		)
-		(property "Footprint" "Capacitor_SMD:C_0402_1005Metric"
+		(property "Footprint" "Capacitor_SMD:C_0603_1608Metric"
 			(at 90.4748 111.76 0)
 			(effects
@@
 			)
 		)
-		(property "Footprint" "Capacitor_SMD:C_0402_1005Metric"
+		(property "Footprint" "Capacitor_SMD:C_0603_1608Metric"
 			(at 76.5048 68.58 0)
 			(effects
@@
 			)
 		)
-		(property "Footprint" "Resistor_SMD:R_0402_1005Metric"
+		(property "Footprint" "Resistor_SMD:R_0805_2012Metric"
 			(at 108.458 72.39 90)
 			(effects
@@
 			)
 		)
-		(property "Datasheet" "https://www.lcsc.com/product-detail/Chip-Resistor-Surface-Mount_UNI-ROYAL-Uniroyal-Elec-0402WGF220KTCE_C25101.html"
+		(property "Datasheet" "https://datasheet.lcsc.com/lcsc/2308241947_FOJAN-FRC0805J270-TS_C2907314.pdf"
 			(at 106.68 72.39 0)
 			(effects
@@
 			)
 		)
-		(property "LCSC" "C25101"
+		(property "LCSC" "C2907304"
 			(at 106.68 72.39 0)
 			(effects
@@
 			)
 		)
-		(property "Footprint" "Capacitor_SMD:C_0402_1005Metric"
+		(property "Footprint" "Capacitor_SMD:C_0603_1608Metric"
 			(at 122.2248 124.46 0)
 			(effects
@@
 			)
 		)
-		(property "Footprint" "Capacitor_SMD:C_0402_1005Metric"
+		(property "Footprint" "Capacitor_SMD:C_0603_1608Metric"
 			(at 166.6748 124.46 0)
 			(effects
@@
 			)
 		)
-		(property "Footprint" "Capacitor_SMD:C_0402_1005Metric"
+		(property "Footprint" "Capacitor_SMD:C_0603_1608Metric"
 			(at 140.0048 124.46 0)
 			(effects
