File: kami.kicad_pcb (KiCad board)
At the start: 4 copper layers, 95 x 86 mm, 119 parts, among them J1 QWIIC, J10 E-Paper, J2 Micro_SD_Card, J3 SAO, J4 EXT, J6 USB-C, J9 Battery, Q2 AP2302B, Q3 AP2302B, Q4 AO3400 (A09T), Q5 AO3400 (A09T), SW6 SW_SPDT, T1 Select, T2 Start, T3 B, T4 A, T5 Cross, T6 Home, T7 Menu, U1 74LVC1G17GW,125, U10 SY6280AAC, U11 SK6805, U12 SK6805, U13 SK6805, U14 SK6805, U15 SK6805, U2 MPR121QR2, U3 ESP32-WROVER-E, U4 TPS63020DSJR, U5 XT4054K421MR-G, U6 SY6280AAC, U7 CH340K, U8 SK6805, U9 SY6280AAC

Commit message: Changes for production version
Parts:
- removed N1: Board, design:board
- C13, C14, C15, C16, C17, C18, C19, C20, C21, C22: footprint Capacitor_SMD:C_0402_1005Metric -> Capacitor_SMD:C_0603_1608Metric
- R34: footprint Resistor_SMD:R_0402_1005Metric -> Resistor_SMD:R_0805_2012Metric
- U6: footprint library:SOT-23-5 -> Package_TO_SOT_SMD:SOT-23-5
- moved C22 2.91 mm to (-32.0, -4.67)
- moved C14 2.47 mm to (-32.0, -6.15)
- moved C21 2.00 mm to (-32.0, -7.62)
- moved C16 1.56 mm to (-32.0, -9.10)
- moved R34 1.51 mm to (-29.2, -20.1)
- moved C20 1.15 mm to (-32.0, -10.6)
- moved D25 1.00 mm to (-39.1, -28.2)
- moved D26 1.00 mm to (-39.1, -26.2)
- moved C18 0.93 mm to (-32.5, -18.7)
- moved C13 0.75 mm to (-36.4, -26.8)
- moved C19 0.73 mm to (-32.0, -12.1)
- moved C17 0.39 mm to (-32.5, -20.2)
- moved R36 0.24 mm to (-32.6, -13.4)
- moved C15 0.08 mm to (-32.5, -14.6)
Routing:
- net GND: track 38.5 -> 35.2 mm, vias 189 -> 188
- net /E-Paper/VCOM: track 3.90 -> 6.91 mm
- net /E-Paper/VSL: track 3.13 -> 5.30 mm
- net /E-Paper/PREVGL: track 22.6 -> 24.8 mm
- net /E-Paper/PREVGH: track 18.8 -> 20.5 mm
- net /E-Paper/VSH: track 2.43 -> 3.29 mm
- net Net-(J10-Pin_7): track 3.82 -> 4.45 mm
Other:
- board text added: "Kami"
- board text added: "Nicolai Electronics"
- board text added: "紙"
- board text removed: "+2025"
- board text removed: "CAUTION: DO NOT LOOK INTO LEDS WITH REMAINING EYE"
- board text removed: "Nicolai Electronics & Badge.Team"
- board text removed: "TSJA"
- board text removed: "Touch me :)"
