File: kami.kicad_sch (KiCad schematic)
At the start: 65 parts, among them J1 QWIIC, J2 Micro_SD_Card, J3 SAO, J4 EXT, J6 USB-C, Q4 AO3400 (A09T), Q5 AO3400 (A09T), T1 Select, T2 Start, T3 B, T4 A, T5 Cross, T6 Home, T7 Menu, U1 74LVC1G17GW,125, U10 SY6280AAC, U11 SK6805, U12 SK6805, U13 SK6805, U14 SK6805, U15 SK6805, U2 MPR121QR2, U3 ESP32-WROVER-E, U7 CH340K, U8 SK6805, U9 SY6280AAC

Commit message: Changes for production version
Other:
- title: TSJA badge -> Kami
Changed lines of the file:
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@@
 (kicad_sch
-	(version 20231120)
+	(version 20250114)
 	(generator "eeschema")
-	(generator_version "8.0")
+	(generator_version "9.0")
 	(paper "A4")
 	(title_block
-		(title "TSJA badge")
-		(date "2024-12-06")
+		(title "Kami")
+		(date "2025-05-20")
 		(rev "1.0")
 		(company "Nicolai Electronics")
 		(comment 1 "License: CERN Open Hardware Licence Version 2 - Permissive")
 	)
+	(rectangle
+		(start 151.13 179.07)
+		(end 176.53 196.85)
+		(stroke
+			(width 0)
+			(type default)
+		)
+		(fill
+			(type none)
+		)
+	)
+	(rectangle
+		(start 140.97 179.07)
+		(end 151.13 196.85)
+		(stroke
+			(width 0)
+			(type default)
+		)
+		(fill
+			(type none)
+		)
+	)
+	(text "Iset: 0.68A\n6800 / 10kOhm"
+		(exclude_from_sim no)
+		(at 82.804 79.248 0)
+		(effects
+			(font
+				(size 0.9906 0.9906)
+			)
+			(justify left bottom)
+		)
+	)
+	(text "M3"
+		(exclude_from_sim no)
+		(at 146.05 181.102 0)
+		(effects
+			(font
+				(size 1.27 1.27)
+			)
+		)
+	)
+	(text "M2"
+		(exclude_from_sim no)
+		(at 163.83 180.848 0)
+		(effects
+			(font
+				(size 1.27 1.27)
+			)
+		)
+	)
+	(text "Iset: 0.68A\n6800 / 10kOhm"
+		(exclude_from_sim no)
+		(at 148.336 23.368 0)
+		(effects
+			(font
+				(size 0.9906 0.9906)
+			)
+			(justify right bottom)
+		)
+	)
+	(text "INPUT ONLY"
+		(exclude_from_sim no)
+		(at 198.628 137.414 0)
+		(effects
+			(font
+				(size 1.27 1.27)
+			)
+			(justify left)
+		)
+	)
+	(text "INPUT ONLY"
+		(exclude_from_sim no)
+		(at 198.628 139.954 0)
+		(effects
+			(font
+				(size 1.27 1.27)
+			)
+			(justify left)
+		)
+	)
 	(junction
 		(at 154.94 111.76)
@@
 		)
 	)
-	(rectangle
-		(start 151.13 179.07)
-		(end 176.53 196.85)
-		(stroke
-			(width 0)
-			(type default)
-		)
-		(fill
-			(type none)
-		)
-	)
-	(rectangle
-		(start 140.97 179.07)
-		(end 151.13 196.85)
-		(stroke
-			(width 0)
-			(type default)
-		)
-		(fill
-			(type none)
-		)
-	)
-	(text "Iset: 0.68A\n6800 / 10kOhm"
-		(exclude_from_sim no)
-		(at 82.804 79.248 0)
-		(effects
-			(font
-				(size 0.9906 0.9906)
-			)
-			(justify left bottom)
-		)
-	)
-	(text "M3"
-		(exclude_from_sim no)
-		(at 146.05 181.102 0)
-		(effects
-			(font
-				(size 1.27 1.27)
-			)
-		)
-	)
-	(text "M2"
-		(exclude_from_sim no)
-		(at 163.83 180.848 0)
-		(effects
-			(font
-				(size 1.27 1.27)
-			)
-		)
-	)
-	(text "Iset: 0.68A\n6800 / 10kOhm"
-		(exclude_from_sim no)
-		(at 148.336 23.368 0)
-		(effects
-			(font
-				(size 0.9906 0.9906)
-			)
-			(justify right bottom)
-		)
-	)
-	(text "INPUT ONLY"
-		(exclude_from_sim no)
-		(at 198.628 137.414 0)
-		(effects
-			(font
-				(size 1.27 1.27)
-			)
-			(justify left)
-		)
-	)
-	(text "INPUT ONLY"
-		(exclude_from_sim no)
-		(at 198.628 139.954 0)
-		(effects
-			(font
-				(size 1.27 1.27)
-			)
-			(justify left)
-		)
-	)
 	(label "CC1"
 		(at 40.64 26.67 0)
-		(fields_autoplaced yes)
 		(effects
 			(font
@@
 	(label "USB_P"
 		(at 44.45 39.37 0)
-		(fields_autoplaced yes)
 		(effects
 			(font
@@
 	(label "USB_N"
 		(at 44.45 36.83 0)
-		(fields_autoplaced yes)
 		(effects
 			(font
@@
 	(label "CC2"
 		(at 40.64 29.21 0)
-		(fields_autoplaced yes)
 		(effects
 			(font
@@
 	(label "USB_VBUS"
 		(at 40.64 21.59 0)
-		(fields_autoplaced yes)
 		(effects
 			(font
@@
 		(at 50.8 56.515)
 		(size 12.7 15.875)
+		(exclude_from_sim no)
+		(in_bom yes)
+		(on_board yes)
+		(dnp no)
 		(fields_autoplaced yes)
 		(stroke
@@
 		)
 		(instances
-			(project "tsja"
+			(project "kami"
 				(path "/5f312b85-6822-40a3-b417-2df49696ca2d"
 					(page "4")
@@
 		(at 64.77 64.77)
 		(size 19.05 7.62)
+		(exclude_from_sim no)
+		(in_bom yes)
+		(on_board yes)
+		(dnp no)
 		(fields_autoplaced yes)
 		(stroke
@@
 		)
 		(instances
-			(project "tsja"
+			(project "kami"
 				(path "/5f312b85-6822-40a3-b417-2df49696ca2d"
 					(page "3")
@@
 		)
 	)
+	(embedded_fonts no)
 )
